File: pcb/mainboard/mainboard.kicad_sch (KiCad schematic)
At the start: 64 parts, among them J1 V_IN, J2 SWD, J3 Conn_01x10, J4 M1, J5 M2, J7 TIP, K1 SANYOU_SRD_Form_C, Q1 NMOS, Q2 NMOS, SW1 RES_BUT, SW2 BOOT_SW, U1 STM32G474RETx, U2 TPS54331DDA, U3 TMC2208_SILENTSTEPSTICK, U4 TMC2208_SILENTSTEPSTICK, U5 INA219AxD, Y1 16MHz

Commit message: Minor Schematic & Major PCB Rework
Parts:
- removed C1, C2, C3, C4, C7: 100n, Capacitor_SMD:C_0603_1608Metric_Pad1.08x0.95mm_HandSolder, symbol Device:C
- removed C10: 4.7u, Capacitor_SMD:C_0603_1608Metric_Pad1.08x0.95mm_HandSolder, symbol Device:C
- removed C11, C9: 1u, Capacitor_SMD:C_0603_1608Metric_Pad1.08x0.95mm_HandSolder, symbol Device:C
- removed C5, C6: 10p, Capacitor_SMD:C_0603_1608Metric_Pad1.08x0.95mm_HandSolder, symbol Device:C
- removed C8: 10n, Capacitor_SMD:C_0603_1608Metric_Pad1.08x0.95mm_HandSolder, symbol Device:C
- removed FB1: 120R, Resistor_SMD:R_0603_1608Metric_Pad0.98x0.95mm_HandSolder, symbol Device:FerriteBead
- removed J2: SWD, CONN_3220-10-0100-00_CNC, symbol CONN_3220-10-0100-00_CNC:3220-10-0100-00
- removed R1, R2: 10k, Resistor_SMD:R_0603_1608Metric_Pad0.98x0.95mm_HandSolder, symbol Device:R
- removed SW1: RES_BUT, Button_Switch_SMD:SW_Tactile_SPST_NO_Straight_CK_PTS636Sx25SMTRLFS, symbol Switch:SW_Push
- removed SW2: BOOT_SW, Button_Switch_THT:SW_Slide_SPDT_Straight_CK_OS102011MS2Q, symbol Switch:SW_SPDT
- removed U1: STM32G474RETx, Package_QFP:LQFP-64_10x10mm_P0.5mm, symbol MCU_ST_STM32G4:STM32G474RETx
- removed Y1: 16MHz, Oscillator:Oscillator_SMD_Abracon_ASE-4Pin_3.2x2.5mm_HandSoldering, symbol Device:Crystal_GND23
- added D2, D4, D5, D6: LED, LED_SMD:LED_0603_1608Metric_Pad1.05x0.95mm_HandSolder, symbol Device:LED
- added D3: D, Diode_SMD:D_0603_1608Metric_Pad1.05x0.95mm_HandSolder, symbol Device:D
- added R12, R13, R14, R16: R, Resistor_SMD:R_0603_1608Metric_Pad0.98x0.95mm_HandSolder, symbol Device:R
- added U6: STM32G474CoreBoard, STM32G474CoreBoard:STM32G474CoreBoard, symbol STM32G474CoreBoard:STM32G474CoreBoard
- C21, C22: footprint (none) -> Capacitor_SMD:CP_Elec_4x4.5
- J3: value Conn_01x10 -> Control Board
Connections:
- net +24V: now also R14.1
- net +3.3V: now also D3.1 (K), R12.1, R13.1
- net +3.3VA: now also U6.1 (VCC), U6.2 (VCC), U6.32 (VREF+)
- net DIR_1: now also U6.18 (PB3)
- net DIR_2: now also U6.20 (PB5)
- net ENC_BTN: now also U6.35 (PA7)
- net ENC_SIG_A: now also U6.10 (PA8)
- net ENC_SIG_B: now also U6.11 (PA9)
- net GND: now also U3.JP2_2 (GND), U3.JP2_8 (GND), D2.1 (K), D5.1 (K), D6.1 (K), U6.27 (GND), U6.28 (GND), U6.3 (GND), U6.4 (GND)
- net INA_SCL: now also U6.15 (PA15)
- net INA_SDA: now also U6.22 (PB7)
- net M1OA1: now also J4.2 (Pin_2); no longer J4.1 (Pin_1)
- net M1OA2: now also J4.1 (Pin_1); no longer J4.2 (Pin_2)
- net M2OA1: now also J5.2 (Pin_2); no longer J5.1 (Pin_1)
- net M2OA2: now also J5.1 (Pin_1); no longer J5.2 (Pin_2)
- net M_ENABLE: now also U6.38 (PA6)
- net OLED_CS: now also U6.40 (PA4)
- net OLED_DC: now also U6.41 (PA1)
- net OLED_MOSI: now also U6.8 (PB15)
- net OLED_RESET: now also U6.44 (PA0)
- net OLED_SCK: now also U6.6 (PB13)
- net STEP_1: now also U6.19 (PB4)
- net STEP_2: now also U6.21 (PB6)
- net TIP_EN: now also R16.1, U6.14 (PA12)
- net V_SELECT: now also U6.16 (PC10)
- net RELAY_OUT: now reaches K1.2, Q1.1 (D)
- net RELAY_OUT: now also D3.2 (A), D4.1 (K)
- net BUCK_3V3_PH: now reaches C16.1, D1.1 (K), L1.1, U2.8 (PH)
- net BUCK_3V3_EN: now reaches R3.1, R4.2, U2.3 (EN)
- net BUCK_3V3_COMP: now reaches C17.1, C18.1, U2.6 (COMP)
- net BUCK_3V3_BOOT: now reaches C16.2, U2.1 (BOOT)
- net BUCK_3V3_SS: now reaches C15.1, U2.4 (SS)
- new net: D5.2 (A), R14.2
- new net: D2.2 (A), R12.2
- new net: D6.2 (A), R16.2
- new net: D4.2 (A), R13.2
- no-connect marks 39 -> 30
Other:
- moved on the sheet: C12, C13, C14, C15, C16, C17, C18, C19, C20, C21, C22, C23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

Commit message: Update PCB
Connections:
- net +3.3VA is gone; now on net +3.3V: U6.1 (VCC), U6.2 (VCC), U6.32 (VREF+)
- net +3.3V: no longer J3.2 (Pin_2)
- net OLED_3V3: now reaches U6.25 (3V3)
- net OLED_3V3: now also J3.2 (Pin_2), U6.26 (3V3)
- no-connect marks 30 -> 28
Changed lines of the file:
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@@
 	)
 	(junction
+		(at 72.39 49.53)
+		(diameter 0)
+		(color 0 0 0 0)
+	)
+	(junction
 		(at 67.31 113.03)
 		(diameter 0)
@@
 	)
 	(no_connect
-		(at 74.93 50.8)
-	)
-	(no_connect
 		(at 264.16 129.54)
 	)
@@
 	)
 	(no_connect
-		(at 72.39 50.8)
-	)
-	(no_connect
 		(at 90.17 64.77)
 	)
@@
 	(wire
 		(pts
+			(xy 72.39 50.8) (xy 72.39 49.53)
+		)
+		(stroke
+			(width 0)
+			(type default)
+		)
+	)
+	(wire
+		(pts
 			(xy 269.24 38.1) (xy 279.4 38.1)
 		)
@@
 	(wire
 		(pts
+			(xy 74.93 50.8) (xy 74.93 49.53)
+		)
+		(stroke
+			(width 0)
+			(type default)
+		)
+	)
+	(wire
+		(pts
+			(xy 72.39 38.1) (xy 77.47 38.1)
+		)
+		(stroke
+			(width 0)
+			(type default)
+		)
+	)
+	(wire
+		(pts
 			(xy 367.03 49.53) (xy 367.03 50.8)
 		)
@@
 	(wire
 		(pts
+			(xy 74.93 49.53) (xy 72.39 49.53)
+		)
+		(stroke
+			(width 0)
+			(type default)
+		)
+	)
+	(wire
+		(pts
 			(xy 138.43 127) (xy 138.43 129.54)
 		)
@@
 	(wire
 		(pts
-			(xy 143.51 45.72) (xy 144.78 45.72)
-		)
-		(stroke
-			(width 0)
-			(type default)
-		)
-	)
-	(wire
-		(pts
 			(xy 251.46 67.31) (xy 262.89 67.31)
 		)
@@
 	(wire
 		(pts
+			(xy 72.39 49.53) (xy 72.39 38.1)
+		)
+		(stroke
+			(width 0)
+			(type default)
+		)
+	)
+	(wire
+		(pts
 			(xy 365.76 49.53) (xy 367.03 49.53)
 		)
@@
 		)
 	)
+	(global_label "OLED_3V3"
+		(shape output)
+		(at 77.47 38.1 0)
+		(fields_autoplaced yes)
+		(effects
+			(font
+				(size 0.889 0.889)
+			)
+			(justify left)
+		)
+		(property "Intersheetrefs" "${INTERSHEET_REFS}"
+			(at 89.708 38.1 0)
+			(effects
+				(font
+					(size 1.27 1.27)
+				)
+				(justify left)
+				(hide yes)
+			)
+		)
+	)
 	(global_label "STEP_2"
 		(shape input)
@@
 		)
 	)
+	(global_label "OLED_3V3"
+		(shape input)
+		(at 144.78 45.72 180)
+		(fields_autoplaced yes)
+		(effects
+			(font
+				(size 0.889 0.889)
+			)
+			(justify right)
+		)
+		(property "Intersheetrefs" "${INTERSHEET_REFS}"
+			(at 132.542 45.72 0)
+			(effects
+				(font
+					(size 1.27 1.27)
+				)
+				(justify right)
+				(hide yes)
+			)
+		)
+	)
 	(global_label "V_SELECT"
 		(shape input)
@@
 			)
 		)
-		(property "Value" "+3.3VA"
+		(property "Value" "+3.3V"
 			(at 64.77 44.704 0)
 			(effects
@@
 	)
 	(symbol
-		(lib_id "power:+3.3V")
-		(at 143.51 45.72 90)
-		(unit 1)
-		(exclude_from_sim no)
-		(in_bom yes)
-		(on_board yes)
-		(dnp no)
-		(property "Reference" "#PWR025"
-			(at 147.32 45.72 0)
-			(effects
-				(font
-					(size 1.27 1.27)
-				)
-				(hide yes)
-			)
-		)
-		(property "Value" "+3.3V"
-			(at 137.922 45.72 90)
-			(effects
-				(font
-					(size 1.27 1.27)
-				)
-			)
-		)
-		(property "Footprint" ""
-			(at 143.51 45.72 0)
-			(effects
-				(font
-					(size 1.27 1.27)
-				)
-				(hide yes)
-			)
-		)
-		(property "Datasheet" ""
-			(at 143.51 45.72 0)
-			(effects
-				(font
-					(size 1.27 1.27)
-				)
-				(hide yes)
-			)
-		)
-		(property "Description" "Power symbol creates a global label with name \"+3.3V\""
-			(at 143.51 45.72 0)
-			(effects
-				(font
-					(size 1.27 1.27)
-				)
-				(hide yes)
-			)
-		)
-		(pin "1"
-		)
-		(instances
-			(project "mainboard"
-				(path "/3cc6bd18-2206-4063-bceb-a55988771b5a"
-					(reference "#PWR025")
-					(unit 1)
-				)
-			)
-		)
-	)
-	(symbol
 		(lib_id "TPS54331DDA:TPS54331DDA")
 		(at 63.5 199.39 0)
@@
 			)
 		)
-		(property "Value" "+3.3VA"
+		(property "Value" "+3.3V"
 			(at 80.01 44.704 0)
 			(effects

Commit message: Update PCB Change Buck Converter Vout  from 3.3V to 5V
Parts:
- removed R6: 0, Resistor_SMD:R_0603_1608Metric_Pad0.98x0.95mm_HandSolder, symbol Device:R
- added R1: 10k, Resistor_SMD:R_0603_1608Metric_Pad0.98x0.95mm_HandSolder, symbol Device:R
- added R2: 1k, Resistor_SMD:R_0603_1608Metric_Pad0.98x0.95mm_HandSolder, symbol Device:R
- D3: value D -> 1N4148-0603
- R12, R13, R16: value R -> 1k
- R14: value R -> 5k
- R7: value 10.2k -> 10k
- R8: value 3.24k -> 1k
Connections:
- net OLED_3V3 is gone; now on net +3.3V: J3.2 (Pin_2), U6.25 (3V3), U6.26 (3V3)
- net +3.3V: no longer C19.1, C20.1, C23.1, C24.1, C25.1, D3.1 (K), K1.4, K1.5, L1.2, R10.1, R12.1, R13.1, R9.1, U3.JP2_7 (VIO), U4.JP2_7 (VIO), U5.5 (VS), U6.1 (VCC), U6.2 (VCC), U6.32 (VREF+)
- net VSENSE: now also R1.2, R2.2; no longer R8.2
- net +5V: now reaches R7.2
- net +5V: now also C19.1, C20.1, C23.1, C24.1, C25.1, D3.1 (K), K1.4, K1.5, L1.2, R10.1, R12.1, R13.1, R9.1, U3.JP2_7 (VIO), U4.JP2_7 (VIO), U5.5 (VS), U6.1 (VCC), U6.2 (VCC), U6.32 (VREF+)
- net BUCK_3V3_BOOT renamed BUCK_5V_BOOT
- net BUCK_3V3_COMP renamed BUCK_5V_COMP
- net BUCK_3V3_EN renamed BUCK_5V_EN
- net BUCK_3V3_PH renamed BUCK_5V_PH
- net BUCK_3V3_SS renamed BUCK_5V_SS
- new net: R1.1, R2.1, R8.2
Other:
- note added: "24V to 5V"
- note removed: "24V to 3.3V"
- moved on the sheet: D3, D4, D6, K1, Q1, Q2, R13, R15, R16, R17, R18, R19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
