File: electronics/mainboard/mainboard.kicad_pcb (KiCad board)
At the start: 2 copper layers, 87.6 x 63.1 mm, 62 parts, among them J1 V_IN, J2 Conn_01x03, J3 Control Board, J4 M1, J5 M2, J6 Conn_01x03, J7 TIP, K1 SANYOU_SRD_Form_C, Q1 NMOS, Q2 NMOS, U2 TPS54331DDA, U3 TMC2208_SILENTSTEPSTICK, U4 TMC2208_SILENTSTEPSTICK, U5 INA219AxD, U6 STM32G474CoreBoard

Commit message: New PCB version
Parts:
- removed JP2: SolderJumper_2_Open, Jumper:SolderJumper-2_P1.3mm_Open_TrianglePad1.0x1.5mm
- removed U6: STM32G474CoreBoard, STM32G474CoreBoard:STM32G474CoreBoard
- added C1: 4.7uF, Capacitor_SMD:C_0805_2012Metric_Pad1.18x1.45mm_HandSolder, F.Cu at (107.2, 71.8)
- added C10: 100nF, Capacitor_SMD:C_0805_2012Metric_Pad1.18x1.45mm_HandSolder, F.Cu at (118.8, 81.8)
- added C11: 100nF, Capacitor_SMD:C_0805_2012Metric_Pad1.18x1.45mm_HandSolder, F.Cu at (118.8, 72.8)
- added C2: 4.7uF, Capacitor_SMD:C_0805_2012Metric_Pad1.18x1.45mm_HandSolder, F.Cu at (113.8, 95.2)
- added C26: 4.7uF, Capacitor_SMD:C_0805_2012Metric_Pad1.18x1.45mm_HandSolder, F.Cu at (114.8, 75.0)
- added C27: 4.7uF, Capacitor_SMD:C_0805_2012Metric_Pad1.18x1.45mm_HandSolder, F.Cu at (114.8, 72.8)
- added C28: 0.01uF, Capacitor_SMD:C_0603_1608Metric_Pad1.08x0.95mm_HandSolder, F.Cu at (148.2, 94.2)
- added C29: 0.01uF, Capacitor_SMD:C_0603_1608Metric_Pad1.08x0.95mm_HandSolder, F.Cu at (148.2, 97.8)
- added C3: 100nF, Capacitor_SMD:C_0805_2012Metric_Pad1.18x1.45mm_HandSolder, F.Cu at (111.5, 95.2)
- added C4: 100nF, Capacitor_SMD:C_0805_2012Metric_Pad1.18x1.45mm_HandSolder, F.Cu at (109.2, 95.2)
- added C5: 12p, Capacitor_SMD:C_0805_2012Metric_Pad1.18x1.45mm_HandSolder, F.Cu at (107.0, 95.2)
- added C6: 12p, Capacitor_SMD:C_0805_2012Metric_Pad1.18x1.45mm_HandSolder, F.Cu at (113.2, 92.0)
- added C7: 100nF, Capacitor_SMD:C_0805_2012Metric_Pad1.18x1.45mm_HandSolder, F.Cu at (118.8, 75.0)
- added C8: 100nF, Capacitor_SMD:C_0805_2012Metric_Pad1.18x1.45mm_HandSolder, F.Cu at (118.8, 77.2)
- added C9: 100nF, Capacitor_SMD:C_0805_2012Metric_Pad1.18x1.45mm_HandSolder, F.Cu at (118.8, 79.5)
- added D7: LED, LED_SMD:LED_0603_1608Metric_Pad1.05x0.95mm_HandSolder, F.Cu at (148.2, 103.0)
- added J8: Conn_ARM_SWD_TagConnect_TC2030-NL, Connector:Tag-Connect_TC2030-IDC-NL_2x03_P1.27mm_Vertical, F.Cu at (124.0, 95.1)
- added JP4: SolderJumper_2_Open, Jumper:SolderJumper-2_P1.3mm_Open_TrianglePad1.0x1.5mm, F.Cu at (147.0, 73.0)
- added L2: 3.3uH, Inductor_SMD:L_Neosid_SMs42, F.Cu at (106.2, 75.8)
- added R2: 1k, Resistor_SMD:R_0603_1608Metric_Pad0.98x0.95mm_HandSolder, F.Cu at (164.2, 95.5)
- added R20: R, Diode_SMD:D_2512_6332Metric_Pad1.52x3.35mm_HandSolder, F.Cu at (144.5, 79.8)
- added R21: 1k, Resistor_SMD:R_0603_1608Metric_Pad0.98x0.95mm_HandSolder, F.Cu at (148.2, 100.8)
- added R6: 33R, Resistor_SMD:R_0805_2012Metric_Pad1.20x1.40mm_HandSolder, F.Cu at (114.8, 77.2)
- added R7: 330m, Diode_SMD:D_2512_6332Metric_Pad1.52x3.35mm_HandSolder, F.Cu at (138.8, 81.0)
- added R8: R, Diode_SMD:D_2512_6332Metric_Pad1.52x3.35mm_HandSolder, F.Cu at (149.2, 79.8)
- added RV1: 10k, Potentiometer_THT:Potentiometer_Vishay_T93YA_Vertical, F.Cu at (153.2, 98.6)
- added U1: RP2350A, RP2350-QFN-60:QFN-60-1EP_7x7mm_P0.4mm_EP3.4x3.4mm_ThermalVias, F.Cu at (111.0, 84.6)
- added U7: LM1117DT-3.3, Package_TO_SOT_SMD:SOT-223-3_TabPin2, F.Cu at (141.8, 94.8)
- added Y1: 12MHz, Crystal:Crystal_SMD_Abracon_ABM8AIG-4Pin_3.2x2.5mm, F.Cu at (109.0, 91.2)
- C21, C22: footprint Capacitor_SMD:CP_Elec_4x4.5 -> Capacitor_SMD:CP_Elec_6.3x7.7
- D3: footprint Diode_SMD:D_0603_1608Metric_Pad1.05x0.95mm_HandSolder -> Diode_SMD:D_1206_3216Metric
- R1: value 10k -> 500R
- R11: value 100 -> 330m; footprint Resistor_SMD:R_1206_3216Metric_Pad1.30x1.75mm_HandSolder -> Diode_SMD:D_2512_6332Metric_Pad1.52x3.35mm_HandSolder
- moved J6 52.5 mm to (127.8, 66.2)
- moved J7 50.8 mm to (138.1, 67.7), turned to 180 degrees
- moved D3 47.2 mm to (167.2, 64.8), turned to 180 degrees
- moved K1 45.4 mm to (154.2, 74.8), turned to 0 degrees
- moved C25 45.0 mm to (125.3, 84.0)
- moved R10 45.0 mm to (126.0, 72.5)
- moved R9 45.0 mm to (127.9, 72.5)
- moved JP3 45.0 mm to (125.9, 88.7)
- moved U5 45.0 mm to (127.9, 78.5)
- moved R15 44.3 mm to (144.5, 64.0)
- moved R17 43.6 mm to (148.8, 64.0), turned to 0 degrees
- moved J2 42.9 mm to (115.2, 66.2)
- moved Q1 42.4 mm to (149.5, 68.2), turned to 0 degrees
- moved D6 41.1 mm to (131.5, 89.3)
- moved R16 41.1 mm to (131.6, 87.7)
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Connections:
- C23 pad 1: +5V -> +3.3V
- C24 pad 1: +5V -> +3.3V
- D3 pad 1: +5V -> +3.3V
- J7 pad 1: TIP_IN -> /ANODE
- JP1 pad 2: +5V -> VBUS
- JP3 pad 1: +5V -> +3.3V
- K1 pad 3: +24V -> VBUS
- K1 pad 4: +5V -> +3.3V
- K1 pad 5: +5V -> +3.3V
- Q1 pad 1: /RELAY_OUT -> Net-(Q1-G)
- Q1 pad 2: Net-(Q1-G) -> GND
- Q1 pad 3: GND -> /RELAY_OUT
- Q2 pad 1: INA- -> Net-(Q2-G)
- Q2 pad 2: Net-(Q2-G) -> GND
- Q2 pad 3: GND -> INA-
- R1 pad 1: Net-(R1-Pad1) -> GND
- R13 pad 1: +5V -> +3.3V
- U3 pad JP1_8: M_ENABLE -> M_ENABLE_1
- U3 pad JP2_7: +5V -> +3.3V
- U4 pad JP1_8: M_ENABLE -> M_ENABLE_2
- U4 pad JP2_7: +5V -> +3.3V
Routing:
- net +3.3V: track 50.7 -> 297.2 mm, vias 0 -> 8
- net +5V: track 160.1 -> 0.00 mm, vias 10 -> 0
- net /uC_VCC: track 66.9 -> 0.00 mm
- net ENC_SIG_B: track 75.6 -> 11.8 mm, vias 1 -> 0
- net ENC_SIG_A: track 67.2 -> 10.2 mm, vias 1 -> 0
- net M_ENABLE: track 56.5 -> 0.00 mm
- net +1.1V: track 0.00 -> 47.7 mm, vias 0 -> 4
- net INA_SCL: track 63.2 -> 18.8 mm, vias 1 -> 2
- net /RELAY_OUT: track 17.3 -> 59.9 mm, vias 0 -> 1
- net M_ENABLE_1: track 0.00 -> 41.3 mm, vias 0 -> 1
- net OLED_SCK: track 49.0 -> 7.94 mm, vias 1 -> 0
- net OLED_MOSI: track 48.2 -> 10.0 mm
- net INA_SDA: track 58.3 -> 20.9 mm, vias 1 -> 2
- net TIP_EN: track 63.8 -> 31.8 mm, vias 0 -> 4
- net VBUS: track 0.00 -> 29.3 mm, vias 0 -> 9
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- added copper zone on F.Cu, net /ANODE
- added copper zone on F.Cu, net INA+
- added copper zone on F.Cu, net TIP_IN
- added copper zone on B.Cu, net VBUS
- added copper zone on F.Cu, net VBUS
- removed copper zone on B.Cu, net +5V
- removed copper zone on F.Cu, net +5V
Other:
- board text added: "3.3V"
- board text added: "CLK"
- board text added: "KN NaMi Tip Etcher v3.0 Adam Matysiak Jakub Klimkowski"
- board text added: "ON OFF VBUS 5V"
- board text added: "RST"
- board text added: "SW1"
- board text added: "SW2"
- board text added: "SWD"
- board text added: "VBUS"
- board text removed: "5V"
- board text removed: "KN NaMi Tip Etcher v1.1 Adam Matysiak Jakub Klimkowski"
- board text removed: "ON OFF 24V 3.3V"
