File: electronics/mainboard/mainboard.kicad_sch (KiCad schematic)
At the start: 61 parts, among them J1 V_IN, J2 Conn_01x03, J3 Control Board, J4 M1, J5 M2, J6 Conn_01x03, J7 TIP, K1 SANYOU_SRD_Form_C, Q1 NMOS, Q2 NMOS, U2 TPS54331DDA, U3 TMC2208_SILENTSTEPSTICK, U4 TMC2208_SILENTSTEPSTICK, U5 INA219AxD, U6 STM32G474CoreBoard

Commit message: New PCB version
Parts:
- added C1: 4.7uF, Capacitor_SMD:C_0805_2012Metric_Pad1.18x1.45mm_HandSolder, symbol Device:C
- added C10, C11, C3, C4, C7, C8, C9: 100nF, Capacitor_SMD:C_0805_2012Metric_Pad1.18x1.45mm_HandSolder, symbol Device:C_Small
- added C2, C26, C27: 4.7uF, Capacitor_SMD:C_0805_2012Metric_Pad1.18x1.45mm_HandSolder, symbol Device:C_Small
- added C28, C29: 0.01uF, Capacitor_SMD:C_0603_1608Metric_Pad1.08x0.95mm_HandSolder, symbol Device:C
- added C5, C6: 12p, Capacitor_SMD:C_0805_2012Metric_Pad1.18x1.45mm_HandSolder, symbol Device:C_Small
- added D7: LED, LED_SMD:LED_0603_1608Metric_Pad1.05x0.95mm_HandSolder, symbol Device:LED
- added J8: Conn_ARM_SWD_TagConnect_TC2030-NL, Connector:Tag-Connect_TC2030-IDC-NL_2x03_P1.27mm_Vertical, symbol Connector:Conn_ARM_SWD_TagConnect_TC2030-NL
- added JP4: SolderJumper_2_Open, Jumper:SolderJumper-2_P1.3mm_Open_TrianglePad1.0x1.5mm, symbol Jumper:SolderJumper_2_Open
- added L2: 3.3uH, Inductor_SMD:L_Neosid_SMs42, symbol Device:L_Small
- added R20: R, Diode_SMD:D_2512_6332Metric_Pad1.52x3.35mm_HandSolder, symbol Device:R
- added R21: 1k, Resistor_SMD:R_0603_1608Metric_Pad0.98x0.95mm_HandSolder, symbol Device:R
- added R6: 33R, Resistor_SMD:R_0805_2012Metric_Pad1.20x1.40mm_HandSolder, symbol Device:R_Small
- added RV1: 10k, Potentiometer_THT:Potentiometer_Vishay_T93YA_Vertical, symbol Device:R_Potentiometer
- added U1: RP2350A, RP2350-QFN-60:QFN-60-1EP_7x7mm_P0.4mm_EP3.4x3.4mm_ThermalVias, symbol rpi-lib-kicad-rp235x:RP2350A
- added U7: LM1117DT-3.3, Package_TO_SOT_SMD:SOT-223-3_TabPin2, symbol Regulator_Linear:LM1117DT-3.3
- added Y1: 12MHz, Crystal:Crystal_SMD_Abracon_ABM8AIG-4Pin_3.2x2.5mm, symbol Device:Crystal_GND24_Small
- C21, C22: footprint Capacitor_SMD:CP_Elec_4x4.5 -> Capacitor_SMD:CP_Elec_6.3x7.7
- D3: footprint Diode_SMD:D_0603_1608Metric_Pad1.05x0.95mm_HandSolder -> Diode_SMD:D_1206_3216Metric
- R1: value 10k -> 500R
- R11: value 100 -> 330m; footprint Resistor_SMD:R_1206_3216Metric_Pad1.30x1.75mm_HandSolder -> Diode_SMD:D_2512_6332Metric_Pad1.52x3.35mm_HandSolder
- R7: value 10k -> 330m; footprint Resistor_SMD:R_0603_1608Metric_Pad0.98x0.95mm_HandSolder -> Diode_SMD:D_2512_6332Metric_Pad1.52x3.35mm_HandSolder
- R8: value 1k -> R; footprint Resistor_SMD:R_0603_1608Metric_Pad0.98x0.95mm_HandSolder -> Diode_SMD:D_2512_6332Metric_Pad1.52x3.35mm_HandSolder
Connections:
- net +24V: now also C28.1, U7.3 (VI); no longer K1.3
- net +3.3V: now also C23.1, C24.1, D3.1 (K), JP3.1 (A), K1.4, K1.5, R13.1, U3.JP2_7 (VIO), U4.JP2_7 (VIO), C10.1, C11.1, C27.1, C29.1, C7.1, C8.1, C9.1, J8.1 (VCC), R21.1, R6.2, U1.1 (IOVDD), U1.11 (IOVDD), U1.20 (IOVDD), U1.30 (IOVDD), U1.38 (IOVDD), U1.44 (ADC_AVDD), U1.45 (IOVDD), U1.49 (VREG_VIN), U1.53 (USB_OTP_VDD), U1.54 (QSPI_IOVDD), U7.2 (VO)
- net +5V: no longer C23.1, C24.1, D3.1 (K), JP1.2 (B), JP3.1 (A), K1.4, K1.5, R13.1, U3.JP2_7 (VIO), U4.JP2_7 (VIO)
- net BUCK_5V_OUT: now also RV1.2, RV1.3; no longer R7.2
- net DIR_1: now also U1.27 (GPIO16)
- net DIR_2: now also U1.29 (GPIO18)
- net ENC_BTN: now also U1.13 (GPIO9)
- net ENC_SIG_A: now also U1.14 (GPIO10)
- net ENC_SIG_B: now also U1.15 (GPIO11)
- net GND: now also Q1.2 (S), Q2.2 (S), R1.1, C1.2, C10.2, C11.2, C2.2, C26.2, C27.2, C28.2, C29.2, C3.2, C4.2, C5.2, C6.2, C7.2, C8.2, C9.2, D7.1 (K), J8.5 (GND), U1.47 (VREG_PGND), U1.61 (GND), U7.1 (GND), Y1.2, Y1.4; no longer Q1.3 (S), Q2.3 (S), R8.1
- net INA+: now also R7.1
- net INA-: now also Q2.3 (D), R7.2; no longer Q2.1 (D)
- net INA_SCL: now also U1.37 (GPIO25)
- net INA_SDA: now also U1.36 (GPIO24)
- net LIMIT_SWITCH_1: now also U1.32 (GPIO20)
- net LIMIT_SWITCH_2: now also U1.33 (GPIO21)
- net M_ENABLE: no longer U3.JP1_8 (EN), U4.JP1_8 (EN)
- net OLED_CS: now also U1.8 (GPIO5)
- net OLED_DC: now also U1.10 (GPIO7)
- net OLED_MOSI: now also U1.5 (GPIO3)
- net OLED_RESET: now also U1.9 (GPIO6)
- net OLED_SCK: now also U1.2 (GPIO0)
- net RELAY_OUT: now also Q1.3 (D); no longer Q1.1 (D)
- net STEP_1: now also U1.28 (GPIO17)
- net STEP_2: now also U1.31 (GPIO19)
- net TIP_EN: now also U1.16 (GPIO12)
- net TIP_IN: now also R8.1, JP4.1 (A); no longer J7.1 (Pin_1)
- net VSENSE: no longer R7.1
- net V_SELECT: now also U1.17 (GPIO13)
- net at R18.2, R19.1: now also Q2.1 (G); no longer Q2.2 (G)
- net at R15.2, R17.1: now also Q1.1 (G); no longer Q1.2 (G)
- new net: R2.1, RV1.1
- new net: C26.1, R6.1, U1.46 (VREG_AVDD)
- new net: C5.1, U1.21 (XIN), Y1.3
- new net: C6.1, U1.22 (XOUT), Y1.1
- new net: J8.4 (SWCLK), U1.24 (SWCLK)
- new net: J8.2 (SWDIO), U1.25 (SWDIO)
- new net: J8.3 (~{RESET}), U1.26 (RUN)
- new net: L2.2, U1.48 (VREG_LX)
- new net: D7.2 (A), R21.2
- new net: R20.1, R8.2
- new net +1.1V: C1.1, C2.1, C3.1, C4.1, L2.1, U1.23 (DVDD), U1.39 (DVDD), U1.50 (VREG_FB), U1.6 (DVDD)
- new net ANODE: J7.1 (Pin_1), JP4.2 (B), R20.2
- new net M_ENABLE_1: U1.19 (GPIO15), U3.JP1_8 (EN)
- new net M_ENABLE_2: U1.18 (GPIO14), U4.JP1_8 (EN)
- new net VBUS: JP1.2 (B), K1.3
- no-connect marks 26 -> 33
Other:
- note added: "24V to 3.3V"
- note added: "24V to adjustable voltage"
- note added: "excluded from board"
- note removed: "24V to 5V"
- moved on the sheet: C12, C13, C14, C15, C16, C17, C18, C19, C20, C21, C22, C23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
